File: baseline_project.kicad_pcb (KiCad board)
At the start: 2 copper layers, 115 x 94 mm, 17 parts, among them J101 EXT_3V3, Q101 IRLD024PBF, SW101 UP, SW102 DOWN, SW103 LEFT, SW104 RIGHT, SW105 MODE, U101 EK-TM4C123GXL, U102 ESP8266-01/ESP-01, U103 Adafruit ST7735R

Commit message: Valvano Dump
Parts:
- removed C102: 100nF, Capacitor_THT:C_Axial_L5.1mm_D3.1mm_P15.00mm_Horizontal
- removed C104: 4.7uF, Capacitor_THT:CP_Axial_L10.0mm_D4.5mm_P15.00mm_Horizontal
- added H1: ~, ECE445L:MountingHole_4_40, F.Cu at (34.9, 121.9)
- added H2: ~, ECE445L:MountingHole_4_40, F.Cu at (34.9, 34.3)
- added H3: ~, ECE445L:MountingHole_4_40, F.Cu at (143.5, 34.3)
- added H4: ~, ECE445L:MountingHole_4_40, F.Cu at (143.5, 121.9)
- added R102: 10k, ECE445L:R_Axial_DIN0204_L3.6mm_D1.6mm_P7.62mm_Horizontal, F.Cu at (82.5, 123.2)
- C101: footprint Capacitor_THT:C_Axial_L5.1mm_D3.1mm_P15.00mm_Horizontal -> ECE445L:C_Axial_200mil
- C103: footprint Capacitor_THT:CP_Axial_L10.0mm_D4.5mm_P15.00mm_Horizontal -> ECE445L:CP_Radial_Tantal200mil
- Q101: footprint footprints:vishay_IRLD024PBF -> ECE445L:DIP920W60P254L490H457Q4N
- R101: footprint Resistor_THT:R_Axial_DIN0411_L9.9mm_D3.6mm_P15.24mm_Horizontal -> ECE445L:R_Axial_DIN0204_L3.6mm_D1.6mm_P7.62mm_Horizontal
- U101: footprint footprints:ti_EKTM4C123GXL -> ECE445L:ti_EKTM4C123GXL
- U102: value ESP8266-01/ESP-01 -> ESP8266-1; footprint footprints:ai_thinker_ESP8266_01 -> ECE445L:PinHeader_2x04_P2.54mm_Vertical
- U103: footprint footprints:adafruit_st7735r -> ECE445L:adafruit_st7735r2
- moved R101 4.17 mm to (143.4, 64.1)
- moved C101 4.11 mm to (142.3, 70.4)
- moved C103 2.64 mm to (142.2, 78.7)
- moved U102 2.21 mm to (135.3, 53.3), turned to -90 degrees
- moved U103 1.89 mm to (104.1, 67.3), turned to 0 degrees
Connections:
- net /SW_DOWN renamed PC7
- net /SW_LEFT renamed PC6
- net /SW_MODE renamed PF4
- net /SW_RIGHT renamed PC5
- net /SW_UP renamed PC4
- Q101 pad 2: /SPEAKER_GATE -> Net-(D101-A)
- Q101 pad 3: GND -> Net-(Q101-G)
- R101 pad 2: Net-(U102-IO0) -> Net-(U102-Ch_PD)
- U101 pad J1_10: /TFT_RST -> PA7
- U101 pad J1_2: unconnected-(U101-PB5-PadJ1_2) -> PB5
- U101 pad J1_3: /SDC_CS -> PB0
- U101 pad J1_4: /SPEAKER_GATE -> PB1
- U101 pad J1_5: /WIFI_TXD -> PE4
- U101 pad J1_6: /WIFI_RXD -> PE5
- U101 pad J1_7: unconnected-(U101-PB4-PadJ1_7) -> PB4
- U101 pad J1_8: /TFT_MOSI -> PA5
- U101 pad J1_9: /TFT_D/C -> PA6
- U101 pad J2_10: /TFT_SCK -> PA2
- U101 pad J2_2: unconnected-(U101-PB2-PadJ2_2) -> PB2
- U101 pad J2_3: /WIFI_IO2 -> PE0
- U101 pad J2_4: unconnected-(U101-PF0-PadJ2_4) -> PF0
- U101 pad J2_6: unconnected-(U101-PB7-PadJ2_6) -> PB7
- U101 pad J2_7: unconnected-(U101-PB6-PadJ2_7) -> PB6
- U101 pad J2_8: /TFT_MISO -> PA4
- U101 pad J2_9: /TFT_CS -> PA3
- U101 pad J3_10: unconnected-(U101-PF1-PadJ3_10) -> PF1
- U101 pad J3_3: unconnected-(U101-PD0-PadJ3_3) -> PD0
- U101 pad J3_4: unconnected-(U101-PD1-PadJ3_4) -> PD1
- U101 pad J3_5: unconnected-(U101-PD2-PadJ3_5) -> PD2
- U101 pad J3_6: unconnected-(U101-PD3-PadJ3_6) -> PD3
- U101 pad J3_7: /~{WIFI_RST} -> PE1
- U101 pad J3_8: unconnected-(U101-PE2-PadJ3_8) -> PE2
- U101 pad J3_9: unconnected-(U101-PE3-PadJ3_9) -> PE3
- U101 pad J4_1: unconnected-(U101-PF2-PadJ4_1) -> PF2
- U101 pad J4_2: unconnected-(U101-PF3-PadJ4_2) -> PF3
- U101 pad J4_3: unconnected-(U101-PB3-PadJ4_3) -> PB3
- U101 pad J4_8: unconnected-(U101-PD6-PadJ4_8) -> PD6
- U101 pad J4_9: unconnected-(U101-PD7-PadJ4_9) -> PD7
- U102 pad 1: GND -> PD7
- U102 pad 2: /WIFI_IO2 -> /WIFI_3V3
- U102 pad 3: Net-(U102-IO0) -> PB4
- U102 pad 4: /WIFI_RXD -> GND
- U102 pad 5: /WIFI_TXD -> PD6
- U102 pad 6: /WIFI_3V3 -> Net-(U102-Ch_PD)
- U102 pad 7: /~{WIFI_RST} -> PB5
- U103 pad 1: +3V3 -> GND
- U103 pad 10: GND -> +3V3
- U103 pad 2: /TFT_MISO -> +3V3
- U103 pad 3: /TFT_SCK -> PA7
- U103 pad 4: /TFT_MOSI -> PA6
- U103 pad 5: /TFT_CS -> PB0
- U103 pad 6: /SDC_CS -> PA3
- U103 pad 7: /TFT_D/C -> PA5
- U103 pad 8: /TFT_RST -> PA2
- U103 pad 9: +3V3 -> PA4
Routing:
- net GND: track 392.9 -> 131.0 mm, vias 1 -> 0
- net +3V3: track 143.8 -> 0.00 mm, vias 4 -> 0
- net /WIFI_RXD: track 113.0 -> 0.00 mm
- net /~{WIFI_RST}: track 105.5 -> 0.00 mm, vias 4 -> 0
- net /WIFI_TXD: track 100.7 -> 0.00 mm, vias 2 -> 0
- net /SPEAKER_GATE: track 100.6 -> 0.00 mm
- net /TFT_RST: track 78.8 -> 0.00 mm, vias 4 -> 0
- net /SDC_CS: track 77.5 -> 0.00 mm, vias 2 -> 0
- net /TFT_D/C: track 76.2 -> 0.00 mm, vias 4 -> 0
- net /TFT_MOSI: track 68.6 -> 0.00 mm, vias 4 -> 0
- net /WIFI_IO2: track 58.3 -> 0.00 mm
- net /WIFI_3V3: track 37.0 -> 0.00 mm
- net /TFT_CS: track 23.8 -> 0.00 mm, vias 2 -> 0
- net Net-(D101-A): track 20.9 -> 0.40 mm
- net /TFT_SCK: track 18.5 -> 0.00 mm, vias 1 -> 0
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Other:
- board text added: "ECE 445L Baseline Project Fall 2024"
- board text removed: "ECE 445L Baseline Project Fall 2023"
