File: baseline_project.kicad_sch (KiCad schematic)
At the start: 17 parts, among them J101 EXT_3V3, Q101 IRLD024PBF, SW101 UP, SW102 DOWN, SW103 LEFT, SW104 RIGHT, SW105 MODE, U101 EK-TM4C123GXL, U102 ESP8266-01/ESP-01, U103 Adafruit ST7735R

Commit message: Valvano Dump
Parts:
- removed C102: 100nF, Capacitor_THT:C_Axial_L5.1mm_D3.1mm_P15.00mm_Horizontal, symbol Device:C_Small
- removed C104: 4.7uF, Capacitor_THT:CP_Axial_L10.0mm_D4.5mm_P15.00mm_Horizontal, symbol Device:C_Polarized_Small_US
- removed U102: ESP8266-01/ESP-01, footprints:ai_thinker_ESP8266_01, symbol ai_thinker_ESP8266_01:ESP8266-01/ESP-01
- removed U103: Adafruit ST7735R, footprints:adafruit_st7735r, symbol adafruit_st7735r:Adafruit ST7735R
- added H1, H2, H3, H4: ~, ECE445L:MountingHole_4_40, symbol ECE445L:MountingHole
- added R102: 10k, ECE445L:R_Axial_DIN0204_L3.6mm_D1.6mm_P7.62mm_Horizontal, symbol ECE445L:R_0.125W
- added U102: ESP8266-1, ECE445L:PinHeader_2x04_P2.54mm_Vertical, symbol ECE445L:ESP8266-1
- added U103: Adafruit ST7735R, ECE445L:adafruit_st7735r2, symbol ECE445L:Adafruit_ST7735R
- C101: footprint Capacitor_THT:C_Axial_L5.1mm_D3.1mm_P15.00mm_Horizontal -> ECE445L:C_Axial_200mil; symbol Device:C_Small -> ECE445L:C
- C103: footprint Capacitor_THT:CP_Axial_L10.0mm_D4.5mm_P15.00mm_Horizontal -> ECE445L:CP_Radial_Tantal200mil; symbol Device:C_Polarized_Small_US -> ECE445L:C_Polarized
- Q101: footprint footprints:vishay_IRLD024PBF -> ECE445L:DIP920W60P254L490H457Q4N; symbol Simulation_SPICE:NMOS -> ECE445L:IRLD024PBF; Height (none) -> 4.57; Manufacturer_Name (none) -> Vishay; Manufacturer_Part_Number (none) -> IRLD024PBF; Mouser Part Number (none) -> 844-IRLD024PBF; Mouser Price/Stock (none) -> https://www.mouser.co.uk/ProductDetail/Vishay-Siliconix/IRL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
- R101: footprint Resistor_THT:R_Axial_DIN0411_L9.9mm_D3.6mm_P15.24mm_Horizontal -> ECE445L:R_Axial_DIN0204_L3.6mm_D1.6mm_P7.62mm_Horizontal; symbol Device:R_Small -> ECE445L:R_0.125W
- U101: footprint footprints:ti_EKTM4C123GXL -> ECE445L:ti_EKTM4C123GXL; symbol ti_EKTM4C123GXL:EK-TM4C123GXL -> ECE445L:EK-TM4C123GXL
Connections:
- net +3V3: now also U103.10 (LITE), U103.2 (VCC)
- net GND: now also Q101.4 (S), U102.4 (GND), U103.1 (GND); no longer Q101.3 (S)
- net WIFI_3V3: now also U102.2 (GPIO0), U102.8 (Vcc)
- net at D101.2 (A), LS101.2, Q101.1 (D): now also Q101.2 (D)
- net PB5: now reaches U101.J1_2 (PB5)
- net PB5: now also U102.7 (Reset)
- net PB4: now reaches U101.J1_7 (PB4)
- net PB4: now also U102.3 (GPIO2)
- net PB2: now reaches U101.J2_2 (PB2)
- net PF0: now reaches U101.J2_4 (PF0)
- net PB7: now reaches U101.J2_6 (PB7)
- net PB6: now reaches U101.J2_7 (PB6)
- net PF1: now reaches U101.J3_10 (PF1)
- net PD0: now reaches U101.J3_3 (PD0)
- net PD1: now reaches U101.J3_4 (PD1)
- net PD2: now reaches U101.J3_5 (PD2)
- net PD3: now reaches U101.J3_6 (PD3)
- net PE2: now reaches U101.J3_8 (PE2)
- net PE3: now reaches U101.J3_9 (PE3)
- net PF2: now reaches U101.J4_1 (PF2)
- net PF3: now reaches U101.J4_2 (PF3)
- net PB3: now reaches U101.J4_3 (PB3)
- net PD6: now reaches U101.J4_8 (PD6)
- net PD6: now also U102.5 (TxD)
- net PD7: now reaches U101.J4_9 (PD7)
- net PD7: now also U102.1 (RxD)
- net at R101.2: now also U102.6 (Ch_PD)
- net SDC_CS renamed PB0
- net PB0: now also U103.5 (CARD_CS)
- net SPEAKER_GATE renamed PB1
- net PB1: now also R102.1; no longer Q101.2 (G)
- net SW_DOWN renamed PC7
- net SW_LEFT renamed PC6
- net SW_MODE renamed PF4
- net SW_RIGHT renamed PC5
- net SW_UP renamed PC4
- net TFT_CS renamed PA3
- net PA3: now also U103.6 (TFT_CS)
- net TFT_D/C renamed PA6
- net PA6: now also U103.4 (D/C)
- net TFT_MISO renamed PA4
- net PA4: now also U103.9 (MISO)
- net TFT_MOSI renamed PA5
- net PA5: now also U103.7 (MOSI)
- net TFT_RST renamed PA7
- net PA7: now also U103.3 (RESET)
- net TFT_SCK renamed PA2
- net PA2: now also U103.8 (SCK)
- net WIFI_IO2 renamed PE0
- net WIFI_RXD renamed PE5
- net WIFI_TXD renamed PE4
- net ~{WIFI_RST} renamed PE1
- new net: Q101.3 (G), R102.2
- no-connect marks 19 -> 1
Other:
- note added: "v1.0.1"
- note added: "v1.0.1 - Fall 2024 revision."
- note removed: "AIN1"
- note removed: "BLUE_LED"
- note removed: "GREEN_LED"
- note removed: "I2C0_SCK"
- note removed: "I2C0_SDA"
- note removed: "PWM0"
- note removed: "RED_LED"
- note removed: "SS1_FS"
- note removed: "SS1_MOSI"
- note removed: "SS1_SCK"
- note removed: "SW2"
- note removed: "TACH"
- note removed: "v1.0.0"
- note removed: "v1.0.0 - Initial revision."
- note removed: "~{RST}"
- moved on the sheet: C101, C103, J101, SW101, SW102, SW103, SW104, SW105
