File: Lab6/Lab6.kicad_sch (KiCad schematic)
At the start: 32 parts, among them J1 JTAG, J2 Battery, SW1 Reset, SW2 Input, U1 TM4C123GH6PMIR, U2 Adafruit ST7735R, U3 LP2950-33LPRE3, Y1 ABM3-16.000MHZ-B2-T

Commit message: Align to grid
Parts:
- removed D2: LED, ECE445L:LED_D5.0mm, symbol ECE445L:LED
- added R3: 10k, ECE445L:R_Axial_DIN0204_L3.6mm_D1.6mm_P7.62mm_Horizontal, symbol ECE445L:R_0.125W
Connections:
- no-connect marks 0 -> 6
Other:
- moved on the sheet: C1, C12, C13, C2, C3, C4, C5, C6, C7, C8, C9, D1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
